Commit message: adjust limits

File: urdf/robot_arm.urdf.xacro (robot description, xacro)
@@ -40,5 +40,5 @@
     <origin xyz="0.047 0 0.135" rpy="0 0 0"/>
     <axis xyz="0 1 0"/>
-    <limit effort="100" velocity="1.5" lower="${-pi/2}" upper="${pi/2}"/>
+    <limit effort="100" velocity="1.5" lower="${-0.42 * pi}" upper="${pi/2}"/>
 </joint>
 <link name="link_2">
@@ -56,5 +56,5 @@
     <origin xyz="0 0 0.110" rpy="0 0 0"/>
     <axis xyz="0 1 0"/>
-    <limit effort="100" velocity="1.5" lower="${-pi/2}" upper="${pi/3}"/>
+    <limit effort="100" velocity="1.5" lower="${-pi/2}" upper="${0.4 * pi}"/>
 </joint>
 <link name="link_3">
@@ -88,5 +88,5 @@
     <origin xyz="0.1175 0 0" rpy="0 0 0"/>
     <axis xyz="0 1 0"/>
-    <limit effort="100" velocity="1.5" lower="${-pi/3}" upper="${pi/3}4"/>
+    <limit effort="100" velocity="1.5" lower="${-0.6 * pi}" upper="${0.6 * pi}"/>
 </joint>
 <link name="link_5">
